File: Usb-BBC.sch (KiCad schematic (older format))
At the start: 24 parts, among them P2 BAT-Connector, P3 BAT-THT, P4 OUT-5V, SW1 SW_SPDT, U2 TP4056, U3 FS312F-G, U4 FS8205, U5 MT3608

Commit message: Serigrafía arreglada.
Parts:
- P1: renamed from P?; footprint (none) -> Connectors_USB:USB_Micro-B_Molex-105017-0001
- P2: footprint (none) -> Connectors_JST:JST_PH_S2B-PH-SM4-TB_02x2.00mm_Angled
- P3, P4: footprint (none) -> Pin_Headers:Pin_Header_Straight_1x02_Pitch2.54mm
- R1, R2, R3, R4, R5, R6, R7: footprint (none) -> Resistors_SMD:R_0603
- SW1: footprint (none) -> Switches:SWITCH_SPST_SMD_A
- U2: footprint (none) -> Housings_SOIC:HTSOP-8-1EP_3.9x4.9mm_Pitch1.27mm_ThermalVias
- U3, U4, U5: footprint (none) -> TO_SOT_Packages_SMD:SOT-23-6
Changed lines of the file:
@@
 F 0 "U2" H 4025 3787 60  0000 C CNN
 F 1 "TP4056" H 4025 3681 60  0000 C CNN
-F 2 "" H 4000 3350 50  0001 C CNN
+F 2 "Housings_SOIC:HTSOP-8-1EP_3.9x4.9mm_Pitch1.27mm_ThermalVias" H 4000 3350 50  0001 C CNN
 F 3 "" H 4000 3350 50  0001 C CNN
 	1    4000 3350
@@
 F 0 "U3" H 5950 4465 50  0000 C CNN
 F 1 "FS312F-G" H 5950 4374 50  0000 C CNN
-F 2 "" H 5900 4050 50  0001 C CNN
+F 2 "TO_SOT_Packages_SMD:SOT-23-6" H 5900 4050 50  0001 C CNN
 F 3 "https://www.ic-fortune.com/upload/Download/FS312F-G-DS-10_EN.pdf" H 5900 4050 50  0001 C CNN
 	1    5950 4050
@@
 F 0 "U5" H 8350 3575 50  0000 C CNN
 F 1 "MT3608" H 8350 3484 50  0000 C CNN
-F 2 "" H 8350 3250 50  0001 C CNN
+F 2 "TO_SOT_Packages_SMD:SOT-23-6" H 8350 3250 50  0001 C CNN
 F 3 "https://www.olimex.com/Products/Breadboarding/BB-PWR-3608/resources/MT3608.pdf" H 8350 3250 50  0001 C CNN
 	1    8350 3250
@@
 F 0 "R1" H 3359 3696 50  0000 L CNN
 F 1 "4k" H 3359 3605 50  0000 L CNN
-F 2 "" H 3300 3650 50  0001 C CNN
+F 2 "Resistors_SMD:R_0603" H 3300 3650 50  0001 C CNN
 F 3 "" H 3300 3650 50  0001 C CNN
 	1    3300 3650
@@
 F 0 "R2" H 4741 3896 50  0000 R CNN
 F 1 "1K" H 4741 3805 50  0000 R CNN
-F 2 "" H 4800 3850 50  0001 C CNN
+F 2 "Resistors_SMD:R_0603" H 4800 3850 50  0001 C CNN
 F 3 "" H 4800 3850 50  0001 C CNN
 	1    4800 3850
@@
 F 0 "R3" H 5009 3896 50  0000 L CNN
 F 1 "1K" H 5009 3805 50  0000 L CNN
-F 2 "" H 4950 3850 50  0001 C CNN
+F 2 "Resistors_SMD:R_0603" H 4950 3850 50  0001 C CNN
 F 3 "" H 4950 3850 50  0001 C CNN
 	1    4950 3850
@@
 F 0 "SW1" V 7004 3248 50  0000 L CNN
 F 1 "SW_SPDT" V 7095 3248 50  0000 L CNN
-F 2 "" H 7050 3100 50  0001 C CNN
+F 2 "Switches:SWITCH_SPST_SMD_A" H 7050 3100 50  0001 C CNN
 F 3 "" H 7050 3100 50  0001 C CNN
 	1    7050 3100
@@
 F 0 "R5" H 5441 4246 50  0000 R CNN
 F 1 "2K" H 5441 4155 50  0000 R CNN
-F 2 "" H 5500 4200 50  0001 C CNN
+F 2 "Resistors_SMD:R_0603" H 5500 4200 50  0001 C CNN
 F 3 "" H 5500 4200 50  0001 C CNN
 	1    5500 4200
@@
 F 0 "U4" H 5950 4435 50  0000 C CNN
 F 1 "FS8205" H 5950 4526 50  0000 C CNN
-F 2 "" H 5950 4800 50  0001 C CNN
+F 2 "TO_SOT_Packages_SMD:SOT-23-6" H 5950 4800 50  0001 C CNN
 F 3 "https://www.ic-fortune.com/upload/Download/FS8205-DS-19_EN.pdf" H 5950 4800 50  0001 C CNN
 	1    5950 4800
@@
 F 0 "R4" V 5250 3800 50  0000 C CNN
 F 1 "100R" V 5400 3650 50  0000 C CNN
-F 2 "" H 5300 3650 50  0001 C CNN
+F 2 "Resistors_SMD:R_0603" H 5300 3650 50  0001 C CNN
 F 3 "" H 5300 3650 50  0001 C CNN
 	1    5300 3650
@@
 F 0 "R6" H 9159 3246 50  0000 L CNN
 F 1 "7.5K" H 9159 3155 50  0000 L CNN
-F 2 "" H 9100 3200 50  0001 C CNN
+F 2 "Resistors_SMD:R_0603" H 9100 3200 50  0001 C CNN
 F 3 "" H 9100 3200 50  0001 C CNN
 	1    9100 3200
@@
 F 0 "R7" H 9159 3546 50  0000 L CNN
 F 1 "1K" H 9159 3455 50  0000 L CNN
-F 2 "" H 9100 3500 50  0001 C CNN
+F 2 "Resistors_SMD:R_0603" H 9100 3500 50  0001 C CNN
 F 3 "" H 9100 3500 50  0001 C CNN
 	1    9100 3500
@@
 F 0 "P2" H 7928 4691 50  0000 L CNN
 F 1 "BAT-Connector" H 7928 4600 50  0000 L CNN
-F 2 "" H 7850 4650 50  0001 C CNN
+F 2 "Connectors_JST:JST_PH_S2B-PH-SM4-TB_02x2.00mm_Angled" H 7850 4650 50  0001 C CNN
 F 3 "" H 7850 4650 50  0001 C CNN
 	1    7850 4650
@@
 F 0 "P4" H 9278 4691 50  0000 L CNN
 F 1 "OUT-5V" H 9278 4600 50  0000 L CNN
-F 2 "" H 9200 4650 50  0001 C CNN
+F 2 "Pin_Headers:Pin_Header_Straight_1x02_Pitch2.54mm" H 9200 4650 50  0001 C CNN
 F 3 "" H 9200 4650 50  0001 C CNN
 	1    9200 4650
@@
 F 0 "P3" H 7928 5091 50  0000 L CNN
 F 1 "BAT-THT" H 7928 5000 50  0000 L CNN
-F 2 "" H 7850 5050 50  0001 C CNN
+F 2 "Pin_Headers:Pin_Header_Straight_1x02_Pitch2.54mm" H 7850 5050 50  0001 C CNN
 F 3 "" H 7850 5050 50  0001 C CNN
 	1    7850 5050
@@
 	6350 6500 6350 6600
 $Comp
-L conn:USB_OTG P?
+L conn:USB_OTG P1
 U 1 1 5C1992D5
 P 2000 3400
-F 0 "P?" V 1575 3324 50  0000 C CNN
+F 0 "P1" V 1575 3324 50  0000 C CNN
 F 1 "USB_OTG" V 1666 3324 50  0000 C CNN
-F 2 "" V 1950 3300 50  0001 C CNN
+F 2 "Connectors_USB:USB_Micro-B_Molex-105017-0001" V 1950 3300 50  0001 C CNN
 F 3 "" V 1950 3300 50  0001 C CNN
 	1    2000 3400
